File: ClockRadio_PhysicalInterface.sch (KiCad schematic (older format))
At the start: 77 parts, among them J1 Interface_tether, SW1 SW_Push, SW2 5WAY_SW, U1 TC1262-33, U2 PCA9685PW

Commit message: Schematic and layout complete
Parts:
- added D1, D3: GRN, LED_SMD:LED_0603_1608Metric_Castellated, symbol Device:LED_Small
- added R1: 120Ω, Resistor_SMD:R_0603_1608Metric, symbol Device:R_Small_US
- added R8: 200Ω, Resistor_SMD:R_0603_1608Metric, symbol Device:R_Small_US
- added TP1, TP2: TestPoint, TestPoint:TestPoint_Pad_D2.0mm, symbol Connector:TestPoint
- renumbered D8 to D10, D1 to D2, D2 to D4, D3 to D5, D4 to D6, D5 to D7, D6 to D8, D7 to D9, R8 to R10, R9 to R11, R10 to R12, R11 to R13, R12 to R14, R13 to R15, R14 to R16, R15 to R17, R16 to R18, R17 to R19, R1 to R2, R18 to R20, R19 to R21, R20 to R22, R21 to R23, R22 to R24, R23 to R25, R24 to R26, R25 to R27, R26 to R28, R27 to R29, R2 to R3, R28 to R30, R29 to R31, R30 to R32, R31 to R33, R32 to R34, R33 to R35, R34 to R36, R35 to R37, R36 to R38, R37 to R39, R3 to R4, R38 to R40, R39 to R41, R40 to R42, R41 to R43, R4 to R5, R5 to R6, R6 to R7, R7 to R9
Connections:
- net GND: now also R1.2, R8.2
- net I2C_SCL: now also J1.2 (Pin_2), R21.2; no longer J1.6 (Pin_6), R20.2
- net I2C_SDA: now also J1.4 (Pin_4), R20.2; no longer J1.5 (Pin_5), R21.2
- net PI_5way: now also J1.6 (Pin_6); no longer J1.1 (Pin_1)
- net PI_pot: now also J1.1 (Pin_1); no longer J1.3 (Pin_3)
- net STBY: now also J1.5 (Pin_5); no longer J1.4 (Pin_4)
- net SYTEM_POWER: now also J1.3 (Pin_3); no longer J1.2 (Pin_2)
- net V3P3: now also R20.1, R21.1, D1.2 (A), TP2.1
- net V6P0: now also D3.2 (A), TP1.1; no longer R20.1, R21.1
- net pot_pullup: now reaches R37.2, RV1.1
- net SW_Right: now reaches R39.1, SW2.4 (RIGHT)
- net SW_Left: now reaches R40.1, SW2.3 (LEFT)
- net SW_Down: now reaches R41.1, SW2.6 (DOWN)
- net SW_UP: now reaches R42.1, SW2.1 (UP)
- net SW_Center: now reaches R43.1, SW2.2 (CENTER)
- new net V3P3_LED: D1.1 (K), R1.1
- new net V6P0_LED: D3.1 (K), R8.1
Other:
- moved on the sheet: J1, R20, R21, R37
